Commit message: Revised launch file for rviz

File: mecademic_description/urdf/meca_500_r3_generated.urdf (robot description, URDF)
Before this commit: robot meca_500_r3, 10 links, 9 joints
Links:
- removed link dummy
- removed link tool0
- added link dummy_meca
- added link tool_meca

File: mecademic_description/urdf/meca_500_r3_macro.xacro (robot description, xacro)
@@ -16,10 +16,4 @@
         </geometry>
       </collision>
-      <inertial>
-        <mass value="1.0"/>
-        <origin rpy="0 0 0" xyz="0 0 0.0"/>
-        <inertia ixx="1.0" iyy="0.0" izz="0.0"
-                ixy="1.0" ixz="0" iyz="1.0"/>
-      </inertial>
     </link>
     <!-- Joint 1 -->
@@ -191,8 +185,8 @@
       <limit effort="10.0" velocity="8.72665" lower="-3.14159" upper="3.14159" />
     </joint>
-    <link name="${prefix}tool0"/>
-    <joint name="${prefix}meca_axis_6_joint-tool0" type="fixed">
+    <link name="${prefix}tool_meca"/>
+    <joint name="${prefix}meca_axis_6_joint-tool_meca" type="fixed">
       <parent link="${prefix}meca_axis_6_link"/>
-      <child link="${prefix}tool0"/>
+      <child link="${prefix}tool_meca"/>
       <origin xyz="0.075 0 0" rpy="0 ${radians(90)} 0"/>
     </joint>
